File: RP2350_80QFN_minimal.kicad_sch (KiCad schematic)
At the start: 49 parts, among them J1 USB_B_Micro, J2 Conn_02x26_Odd_Even, J3 Conn_02x26_Odd_Even, J4 SM03B-SRSS-TB, SW1 SW_Push, SW2 SW_Push, U1 RP2350_80QFN, U2 NCP1117-3.3_SOT223, U3 W25Q128JVS, U4 DNF, Y1 ABM8-272-T3

Commit message: added jlcpcb part numbers, configured do-not-pop
Primary flash is configured as secondary.
Through-hole connectors not populated.
Parts:
- C1, C19, C5: LCSC PN (none) -> C15850
- C10, C6, C7, C9: LCSC PN (none) -> C368809
- C11, C12, C13, C14, C15, C16, C17, C18, C2, C20, C21, C8: LCSC PN (none) -> C16193311
- C22, H1, H2, H3, H4, J2, J3, R10, R11, R13, U4: now not fitted; now left out of the parts list
- C3, C4: LCSC PN (none) -> C307341
- J1: LCSC PN (none) -> C428495
- J4: LCSC PN (none) -> C160403
- L1: LCSC PN (none) -> C42411119
- R1: value DNF -> 10k; LCSC PN (none) -> C25744
- R2, R4, R6: LCSC PN (none) -> C11702
- R3: LCSC PN (none) -> C25105
- R7, R8: LCSC PN (none) -> C138021
- R9: value DNF -> 0; LCSC PN (none) -> C17168
- SW1, SW2: LCSC PN (none) -> C115360
- U1: LCSC PN (none) -> C39843328
- U2: LCSC PN (none) -> C26537
- U3: LCSC PN (none) -> C97521
- Y1: LCSC PN (none) -> C20625731
