File: RP2350_80QFN_minimal.kicad_sch (KiCad schematic)
At the start: 49 parts, among them J1 USB_B_Micro, J2 Conn_02x26_Odd_Even, J3 Conn_02x26_Odd_Even, J4 SM03B-SRSS-TB, SW1 SW_Push, SW2 SW_Push, U1 RP2350_80QFN, U2 NCP1117-3.3_SOT223, U3 W25Q128JVS, U4 DNF, Y1 ABM8-272-T3

Commit message: added USB-C to the board.
Parts:
- removed J1: USB_B_Micro, Connector_USB:USB_Micro-B_Amphenol_10103594-0001LF_Horizontal, symbol Connector:USB_B_Micro
- added J5: USB_C_Receptacle_USB2.0_16P, Connector_USB:USB_C_Receptacle_HRO_TYPE-C-31-M-12, symbol Connector:USB_C_Receptacle_USB2.0_16P
- added R12, R5: 5k1, Resistor_SMD:R_0805_2012Metric_Pad1.20x1.40mm_HandSolder, symbol Device:R
- added U5: USBLC6-2SC6, Package_TO_SOT_SMD:SOT-23-6, symbol Power_Protection:USBLC6-2SC6
Connections:
- net GND: now also J5.A1 (GND), J5.A12 (GND), J5.B1 (GND), J5.B12 (GND), J5.SH (SHIELD), R12.2, R5.2, U5.2 (GND)
- net USB_D+: now also U5.4 (I/O2)
- net USB_D-: now also U5.6 (I/O1)
- net VBUS: now also J5.A4 (VBUS), J5.A9 (VBUS), J5.B4 (VBUS), J5.B9 (VBUS), U5.5 (VBUS)
- new net CC1: J5.A5 (CC1), R12.1
- new net CC2: J5.B5 (CC2), R5.1
- new net D+: J5.A6 (D+), J5.B6 (D+), U5.3 (I/O2)
- new net D-: J5.A7 (D-), J5.B7 (D-), U5.1 (I/O1)
- no-connect marks 1 -> 2
Other:
- note added: "500mA - 3A @ 5V"
- moved on the sheet: C1, C5, U2
