File: RP2350_80QFN_minimal.kicad_pcb (KiCad board)
At the start: 2 copper layers, 52 x 71.5 mm, 49 parts, among them J1 USB_B_Micro, J2 Conn_02x26_Odd_Even, J3 Conn_02x26_Odd_Even, J4 SM03B-SRSS-TB, SW1 SW_Push, SW2 SW_Push, U1 RP2350_80QFN, U2 NCP1117-3.3_SOT223, U3 W25Q128JVS, U4 DNF, Y1 ABM8-272-T3

Commit message: as submitted to jlcpcb for manufacturing
Parts:
- R1: value DNF -> 10k
- R9: value DNF -> 0
Other:
- rule pad_to_mask_clearance: 0.03 -> 0
