File: RP2350_80QFN_minimal.kicad_pcb (KiCad board)
At the start: 2 copper layers, 52 x 71.5 mm, 49 parts, among them J1 USB_B_Micro, J2 Conn_02x26_Odd_Even, J3 Conn_02x26_Odd_Even, J4 SM03B-SRSS-TB, SW1 SW_Push, SW2 SW_Push, U1 RP2350_80QFN, U2 NCP1117-3.3_SOT223, U3 W25Q128JVS, U4 DNF, Y1 ABM8-272-T3

Commit message: added USB-C to the board.
Parts:
- removed J1: USB_B_Micro, Connector_USB:USB_Micro-B_Amphenol_10103594-0001LF_Horizontal
- added J5: USB_C_Receptacle_USB2.0_16P, Connector_USB:USB_C_Receptacle_HRO_TYPE-C-31-M-12, F.Cu at (99.0, 72.2)
- added R12: 5k1, Resistor_SMD:R_0805_2012Metric_Pad1.20x1.40mm_HandSolder, F.Cu at (103.0, 80.0)
- added R5: 5k1, Resistor_SMD:R_0805_2012Metric_Pad1.20x1.40mm_HandSolder, F.Cu at (95.0, 80.0)
- added U5: USBLC6-2SC6, Package_TO_SOT_SMD:SOT-23-6, F.Cu at (99.0, 80.2)
- moved C5 3.42 mm to (109.4, 92.4)
- moved C1 3.27 mm to (108.3, 79.5)
- moved U2 3.27 mm to (108.4, 85.6)
- moved C2 0.97 mm to (96.2, 83.8)
Routing:
- net VBUS: track 2.11 -> 25.6 mm, vias 0 -> 4
- net /D+: track 0.00 -> 11.1 mm
- net /D-: track 0.00 -> 8.03 mm, vias 0 -> 2
- net /USB_D-: track 16.3 -> 9.74 mm
- net /CC1: track 0.00 -> 6.48 mm
- net /USB_D+: track 16.4 -> 10.1 mm
- net /CC2: track 0.00 -> 6.27 mm
- net GND: track 38.8 -> 38.7 mm, vias 29 -> 31
- removed copper zone on F.Cu, net VBUS
Other:
- board text added: "Minimal Design Example REV3.1"
- board text removed: "Minimal Design Example REV3"

Commit message: added cool symbols!
Parts:
- added REF**: KiCad-Logo_8mm_SilkScreen, Symbol:KiCad-Logo_8mm_SilkScreen, B.Cu at (108.8, 82.8)
Other:
- board text added: "jdfin, Tk"
